File: pg_hw/pg_hw.kicad_sch (KiCad schematic)
At the start: 0 parts

Commit message: Add some libarry
ad some library
Other:
- added sheet BMS (BMS.kicad_sch)
- added sheet Boost (Boost.kicad_sch)
Changed lines of the file:
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@@
 	(paper "A4")
 	(sheet
+		(at 238.76 43.18)
+		(size 19.05 19.05)
+		(fields_autoplaced yes)
+		(stroke
+			(width 0.1524)
+			(type solid)
+		)
+		(fill
+			(color 0 0 0 0.0000)
+		)
+		(property "Sheetname" "BMS"
+			(at 238.76 42.4684 0)
+			(effects
+				(font
+					(size 1.27 1.27)
+				)
+				(justify left bottom)
+			)
+		)
+		(property "Sheetfile" "BMS.kicad_sch"
+			(at 238.76 62.8146 0)
+			(effects
+				(font
+					(size 1.27 1.27)
+				)
+				(justify left top)
+			)
+		)
+		(instances
+			(project "pg_hw"
+				(path "/98c2be80-c7ca-4fe5-b302-238a0f594199"
+					(page "5")
+				)
+			)
+		)
+	)
+	(sheet
 		(at 158.75 40.64)
-		(size 38.1 19.05)
+		(size 19.05 16.51)
 		(fields_autoplaced yes)
 		(stroke
@@
 		)
 		(property "Sheetfile" "LCD.kicad_sch"
-			(at 158.75 60.2746 0)
+			(at 158.75 57.7346 0)
 			(effects
 				(font
@@
 				)
 			)
+		)
+	)
+	(sheet
+		(at 199.39 40.64)
+		(size 27.94 17.78)
+		(fields_autoplaced yes)
+		(stroke
+			(width 0.1524)
+			(type solid)
+		)
+		(fill
+			(color 0 0 0 0.0000)
+		)
+		(property "Sheetname" "Boost"
+			(at 199.39 39.9284 0)
+			(effects
+				(font
+					(size 1.27 1.27)
+				)
+				(justify left bottom)
+			)
+		)
+		(property "Sheetfile" "Boost.kicad_sch"
+			(at 199.39 59.0046 0)
+			(effects
+				(font
+					(size 1.27 1.27)
+				)
+				(justify left top)
+			)
+		)
+		(instances
+			(project "pg_hw"
+				(path "/98c2be80-c7ca-4fe5-b302-238a0f594199"
+					(page "4")
+				)
+			)
