File: pg_hw/controller.kicad_sch (KiCad schematic)
At the start: 27 parts, among them J1 USB_C_Receptacle_USB2.0_14P, J2 Conn_01x03_Pin, J3 Conn_01x03_Pin, Q1 SS8050, Q2 SS8050, SW1 SW_MEC_5E, SW2 SW_MEC_5E, U1 BW16, U2 AMS1117-3.3, U3 CH340C

Commit message: update some things
Parts:
- R1, R2, R3, R4, R5, R6: footprint (none) -> Resistor_SMD:R_0603_1608Metric
- U1: footprint BW16:MODULE_BW16 -> footprints:MODULE_BW16
Changed lines of the file:
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@@
 			)
 		)
-		(property "Footprint" ""
+		(property "Footprint" "Resistor_SMD:R_0603_1608Metric"
 			(at 167.894 30.734 90)
 			(effects
@@
 			)
 		)
-		(property "Footprint" ""
+		(property "Footprint" "Resistor_SMD:R_0603_1608Metric"
 			(at 55.626 118.364 90)
 			(effects
@@
 			)
 		)
-		(property "Footprint" ""
+		(property "Footprint" "Resistor_SMD:R_0603_1608Metric"
 			(at 63.754 35.814 90)
 			(effects
@@
 			)
 		)
-		(property "Footprint" ""
+		(property "Footprint" "Resistor_SMD:R_0603_1608Metric"
 			(at 166.624 47.244 90)
 			(effects
@@
 			)
 		)
-		(property "Footprint" ""
+		(property "Footprint" "Resistor_SMD:R_0603_1608Metric"
 			(at 63.754 38.354 90)
 			(effects
@@
 			)
 		)
-		(property "Footprint" ""
+		(property "Footprint" "Resistor_SMD:R_0603_1608Metric"
 			(at 55.626 141.224 90)
 			(effects
@@
 			)
 		)
-		(property "Footprint" "BW16:MODULE_BW16"
+		(property "Footprint" "footprints:MODULE_BW16"
 			(at 119.38 71.12 0)
 			(effects

Commit message: change batt again
Parts:
- added R7, R8: R_US, symbol Device:R_US
- D5: footprint Diode_THT:D_DO-41_SOD81_P10.16mm_Horizontal -> Diode_SMD:Nexperia_CFP3_SOD-123W
- U3: footprint Package_SO:SOIC-16_3.9x9.9mm_P1.27mm -> Package_SO:SOP-16_3.9x9.9mm_P1.27mm
Connections:
- net +3V3: now also R7.1, R8.1
- net PA25 renamed LP_I2C_SCL
- net LP_I2C_SCL: now also R7.2
- net PA26 renamed LP_I2C_SDA
- net LP_I2C_SDA: now also R8.2

Commit message: hui
Parts:
- C1, C2, C3, C4: footprint (none) -> Resistor_SMD:R_0603_1608Metric
- D5: footprint Diode_SMD:Nexperia_CFP3_SOD-123W -> Diode_THT:D_DO-41_SOD81_P10.16mm_Horizontal
- R3, R4, R5, R6: footprint Resistor_SMD:R_0603_1608Metric -> Resistor_SMD:R_0402_1005Metric
- R7, R8: footprint (none) -> Resistor_SMD:R_0402_1005Metric
Changed lines of the file:
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@@
 			)
 		)
-		(property "Footprint" "Resistor_SMD:R_0603_1608Metric"
+		(property "Footprint" "Resistor_SMD:R_0402_1005Metric"
 			(at 167.894 30.734 90)
 			(effects
@@
 			)
 		)
-		(property "Footprint" ""
+		(property "Footprint" "Resistor_SMD:R_0603_1608Metric"
 			(at 127.9652 40.64 0)
 			(effects
@@
 			)
 		)
-		(property "Footprint" "Resistor_SMD:R_0603_1608Metric"
+		(property "Footprint" "Resistor_SMD:R_0402_1005Metric"
 			(at 55.626 118.364 90)
 			(effects
@@
 			)
 		)
-		(property "Footprint" ""
+		(property "Footprint" "Resistor_SMD:R_0603_1608Metric"
 			(at 92.4052 40.64 0)
 			(effects
@@
 			)
 		)
-		(property "Footprint" "Diode_SMD:Nexperia_CFP3_SOD-123W"
+		(property "Footprint" "Diode_THT:D_DO-41_SOD81_P10.16mm_Horizontal"
 			(at 46.99 126.365 0)
 			(effects
@@
 			)
 		)
-		(property "Footprint" ""
+		(property "Footprint" "Resistor_SMD:R_0402_1005Metric"
 			(at 178.816 66.294 90)
 			(effects
@@
 			)
 		)
-		(property "Footprint" "Resistor_SMD:R_0603_1608Metric"
+		(property "Footprint" "Resistor_SMD:R_0402_1005Metric"
 			(at 166.624 47.244 90)
 			(effects
@@
 			)
 		)
-		(property "Footprint" ""
+		(property "Footprint" "Resistor_SMD:R_0603_1608Metric"
 			(at 121.6152 40.64 0)
 			(effects
@@
 			)
 		)
-		(property "Footprint" "Resistor_SMD:R_0603_1608Metric"
+		(property "Footprint" "Resistor_SMD:R_0402_1005Metric"
 			(at 55.626 141.224 90)
 			(effects
@@
 			)
 		)
-		(property "Footprint" ""
+		(property "Footprint" "Resistor_SMD:R_0402_1005Metric"
 			(at 169.926 66.294 90)
 			(effects
@@
 			)
 		)
-		(property "Footprint" ""
+		(property "Footprint" "Resistor_SMD:R_0603_1608Metric"
 			(at 100.0252 40.64 0)
 			(effects

Commit message: push
Parts:
- added U7: PCF8574A, symbol Interface_Expansion:PCF8574A
- R7, R8: value R_US -> 10K
Connections:
- net +3V3: now also U7.16 (VDD)
- net +5V: no longer C1.1, C2.1, U2.3 (VI)
- net GND: now also U7.8 (VSS)
- net LP_I2C_SCL: now also U7.14 (SCL), U7.15 (SDA)
- new net 4.2V: C1.1, C2.1, U2.3 (VI)
Other:
- moved on the sheet: D3

Commit message: ADD REV
DADA
Connections:
- net GND: now also U7.1 (A0), U7.2 (A1), U7.3 (A2)
- net LP_I2C_SCL: no longer U7.15 (SDA)
- net LP_I2C_SDA: now also U7.15 (SDA)
- net PA8_RX: now also U7.13 (~{INT})
- net Q_touch_5: now reaches U7.10 (P5)
- net Q_touch_1: now reaches U7.5 (P1)
- net Q_touch_2: now reaches U7.6 (P2)
- net Q_touch_3: now reaches U7.7 (P3)
- net Q_touch_4: now reaches U7.9 (P4)
- net PA27 renamed LED_LCD
- net PA30 renamed LCD_RESET
- net PA7_TX renamed BUZZER
- net PB3 renamed LCD_DC

Commit message: Mungkin masih akan ada refisi
munvkin
Parts:
- removed J2, J3: Conn_01x03_Pin, symbol Connector:Conn_01x03_Pin
- added R30, R31, R32, R33, R34: 0, symbol Device:R
Connections:
- net BUZZER: now also U7.4 (P0), R34.2; no longer Q2.3 (C), SW2.1, SW2.2, U1.11 (PA7)
- net CH340_RX0: now also R32.1, R33.2
- net PA8_RX: now also R31.2
- net PB1_TXD: now also R32.2
- net PB2_RXD: now also R30.1
- net CTP_RST: now reaches U7.11 (P6)
- net CTP_INT: now reaches U7.12 (P7)
- net at D4.2 (A): now also R30.2, R31.1
- net LP_I2C_SCL renamed CTP_SCL
- net LP_I2C_SDA renamed CTP_SDA
- new net PA7_TX: Q2.3 (C), R33.1, R34.1, SW2.1, SW2.2
Other:
- moved on the sheet: D4, D6, R6

Commit message: charlotte andeh
charlotte andeh
Parts:
- added R35: 10K, Resistor_SMD:R_0402_1005Metric, symbol Device:R_US
Connections:
- net Q_touch_5 is gone; now on net LED_LCD: U7.10 (P5)
- net +3V3: now also R35.1
- net LED_LCD: no longer U1.6 (PA27)
- net PA8_RX: no longer U1.5 (PA8), U7.13 (~{INT})
- new net PA27: R35.2, U1.6 (PA27), U7.13 (~{INT})
Changed lines of the file:
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@@
 	)
 	(junction
+		(at 177.8 130.81)
+		(diameter 0)
+		(color 0 0 0 0)
+	)
+	(junction
 		(at 177.8 60.96)
 		(diameter 0)
@@
 	(wire
 		(pts
-			(xy 137.16 76.2) (xy 172.72 76.2)
+			(xy 137.16 76.2) (xy 153.67 76.2)
 		)
 		(stroke
@@
 	(wire
 		(pts
-			(xy 213.36 130.81) (xy 73.66 130.81)
-		)
-		(stroke
-			(width 0)
-			(type default)
-		)
-	)
-	(wire
-		(pts
 			(xy 201.93 45.72) (xy 215.9 45.72)
 		)
@@
 	(wire
 		(pts
-			(xy 73.66 130.81) (xy 73.66 68.58)
-		)
-		(stroke
-			(width 0)
-			(type default)
-		)
-	)
-	(wire
-		(pts
 			(xy 210.82 118.11) (xy 213.36 118.11)
 		)
@@
 	(wire
 		(pts
+			(xy 180.34 118.11) (xy 177.8 118.11)
+		)
+		(stroke
+			(width 0)
+			(type default)
+		)
+	)
+	(wire
+		(pts
 			(xy 93.98 109.22) (xy 100.33 109.22)
 		)
@@
 	(wire
 		(pts
-			(xy 238.76 123.19) (xy 245.11 123.19)
+			(xy 238.76 123.19) (xy 246.38 123.19)
 		)
 		(stroke
@@
 	(wire
 		(pts
+			(xy 177.8 128.27) (xy 177.8 130.81)
+		)
+		(stroke
+			(width 0)
+			(type default)
+		)
+	)
+	(wire
+		(pts
 			(xy 54.61 152.4) (xy 54.61 157.48)
 		)
@@
 	(wire
 		(pts
-			(xy 96.52 99.06) (xy 93.98 99.06)
+			(xy 153.67 130.81) (xy 153.67 76.2)
 		)
 		(stroke
@@
 	(wire
 		(pts
-			(xy 54.61 140.97) (xy 54.61 144.78)
+			(xy 96.52 99.06) (xy 93.98 99.06)
 		)
 		(stroke
@@
 	(wire
 		(pts
-			(xy 73.66 68.58) (xy 101.6 68.58)
+			(xy 54.61 140.97) (xy 54.61 144.78)
 		)
 		(stroke
@@
 	(wire
 		(pts
+			(xy 177.8 118.11) (xy 177.8 120.65)
+		)
+		(stroke
+			(width 0)
+			(type default)
+		)
+	)
+	(wire
+		(pts
 			(xy 109.22 43.18) (xy 120.65 43.18)
 		)
@@
 	(wire
 		(pts
+			(xy 177.8 130.81) (xy 153.67 130.81)
+		)
+		(stroke
+			(width 0)
+			(type default)
+		)
+	)
+	(wire
+		(pts
 			(xy 181.61 25.4) (xy 181.61 26.67)
 		)
@@
 	(wire
 		(pts
+			(xy 213.36 130.81) (xy 177.8 130.81)
+		)
+		(stroke
+			(width 0)
+			(type default)
+		)
+	)
+	(wire
+		(pts
 			(xy 171.45 31.75) (xy 173.99 31.75)
 		)
@@
 		)
 	)
-	(global_label "Q_touch_5"
-		(shape input)
-		(at 245.11 123.19 0)
-		(fields_autoplaced yes)
-		(effects
-			(font
-				(size 1.27 1.27)
-			)
-			(justify left)
-		)
-		(property "Intersheetrefs" "${INTERSHEET_REFS}"
-			(at 257.8317 123.19 0)
-			(effects
-				(font
-					(size 1.27 1.27)
-				)
-				(justify left)
-				(hide yes)
-			)
-		)
-	)
 	(global_label "CTP_INT"
 		(shape input)
@@
 	(global_label "LED_LCD"
 		(shape input)
-		(at 172.72 76.2 0)
+		(at 246.38 123.19 0)
 		(fields_autoplaced yes)
 		(effects
@@
 		)
 		(property "Intersheetrefs" "${INTERSHEET_REFS}"
-			(at 183.688 76.2 0)
+			(at 257.348 123.19 0)
 			(effects
 				(font
@@
 	)
 	(symbol
+		(lib_id "Device:R_US")
+		(at 177.8 124.46 0)
+		(unit 1)
+		(exclude_from_sim no)
+		(in_bom yes)
+		(on_board yes)
+		(dnp no)
+		(property "Reference" "R35"
+			(at 177.8 120.904 0)
+			(effects
+				(font
+					(size 1.27 1.27)
+				)
+				(justify left)
+			)
+		)
+		(property "Value" "10K"
+			(at 178.054 128.016 0)
+			(effects
+				(font
+					(size 1.27 1.27)
+				)
+				(justify left)
+			)
+		)
+		(property "Footprint" "Resistor_SMD:R_0402_1005Metric"
+			(at 178.816 124.714 90)
+			(effects
+				(font
+					(size 1.27 1.27)
+				)
+				(hide yes)
+			)
+		)
+		(property "Datasheet" "~"
+			(at 177.8 124.46 0)
+			(effects
+				(font
+					(size 1.27 1.27)
+				)
+				(hide yes)
+			)
+		)
+		(property "Description" "Resistor, US symbol"
+			(at 177.8 124.46 0)
+			(effects
+				(font
+					(size 1.27 1.27)
+				)
+				(hide yes)
+			)
+		)
+		(pin "1"
+		)
+		(pin "2"
+		)
+		(instances
+			(project "pg_hw"
+				(path "/98c2be80-c7ca-4fe5-b302-238a0f594199/8ba1f843-15ae-42f6-a267-5fa0b50da669"
+					(reference "R35")
+					(unit 1)
+				)
+			)
+		)
+	)
+	(symbol
 		(lib_id "Device:C")
 		(at 91.44 36.83 0)
@@
 					(unit 1)
 				)
+			)
+		)
+	)
+	(symbol
+		(lib_id "power:+3V3")
+		(at 180.34 118.11 270)
+		(unit 1)
+		(exclude_from_sim no)
+		(in_bom yes)
+		(on_board yes)
+		(dnp no)
+		(fields_autoplaced yes)
+		(property "Reference" "#PWR050"
+			(at 176.53 118.11 0)
+			(effects
+				(font
+					(size 1.27 1.27)
+				)
+				(hide yes)
+			)
+		)
+		(property "Value" "+3V3"
+			(at 184.15 118.1099 90)
+			(effects
+				(font
+					(size 1.27 1.27)
+				)
+				(justify left)
+			)
+		)
+		(property "Footprint" ""
+			(at 180.34 118.11 0)
+			(effects
+				(font
+					(size 1.27 1.27)
+				)
+				(hide yes)
+			)
+		)
+		(property "Datasheet" ""
+			(at 180.34 118.11 0)
+			(effects
+				(font
+					(size 1.27 1.27)
+				)
+				(hide yes)
+			)
+		)
+		(property "Description" "Power symbol creates a global label with name \"+3V3\""
+			(at 180.34 118.11 0)
+			(effects
+				(font
+					(size 1.27 1.27)
+				)
+				(hide yes)
+			)
+		)
+		(pin "1"
+		)
+		(instances
+			(project "pg_hw"
+				(path "/98c2be80-c7ca-4fe5-b302-238a0f594199/8ba1f843-15ae-42f6-a267-5fa0b50da669"
+					(reference "#PWR050")
+					(unit 1)
+				)

Commit message: usb revision
add some revision
Parts:
- removed J1: USB_C_Receptacle_USB2.0_14P, symbol Connector:USB_C_Receptacle_USB2.0_14P
- removed R1, R2: 5.1K, Resistor_SMD:R_0603_1608Metric, symbol Device:R_US
- added J1: USB_B_Micro, symbol Connector:USB_B_Micro
Connections:
- net GND: now also J1.5 (GND), J1.6 (Shield)
- net VBUS: now also J1.1 (VBUS)
- net usb_d+: now also J1.3 (D+)
- net usb_d-: now also J1.2 (D-)
