File: pg_hw/controller.kicad_sch (KiCad schematic)
At the start: 32 parts, among them J1 USB_B_Micro, Q1 SS8050, Q2 SS8050, SW1 SW_MEC_5E, SW2 SW_MEC_5E, U1 BW16, U2 AMS1117-3.3, U3 CH340C, U7 PCF8574A

Commit message: adad
dada
Parts:
- removed D1, D3, D4, D5, D6: 1N5819, Diode_THT:D_DO-41_SOD81_P10.16mm_Horizontal, symbol Diode:1N5819
- added D1, D4, D5, D8, D9: SS14, Diode_SMD:D_SMA, symbol Diode:SS14
- C1, C2, C3, C4: footprint Resistor_SMD:R_0603_1608Metric -> Capacitor_SMD:C_0603_1608Metric
- C5: footprint (none) -> Capacitor_SMD:C_0603_1608Metric
- J1: footprint (none) -> Connector_USB:USB_Micro-B_Molex-105017-0001
- R30, R31, R32, R33, R34: footprint (none) -> Resistor_SMD:R_0402_1005Metric
Connections:
- net +5V: now also D4.1 (K)
- net CH340_TXD: now also D9.1 (K)
- net PA8_LOG_RX: now also D1.1 (K), D8.1 (K)
- net PA8_RX: now also D1.2 (A), D8.2 (A)
- net PB2_RXD: now also D5.2 (A)
- net RXD: now also D5.1 (K)
- net VBUS: now also D4.2 (A)
- net at R30.2, R31.1: now also D9.2 (A)
