File: pg_hw/Boost.kicad_sch (KiCad schematic)
At the start: 1 part, among them U5 TPS61088RHLR

Commit message: updarte schematics
schematics menuju pengecheckan
Parts:
- added C10, C11, C12: 47nF, symbol Device:C
- added C13: 1uF, symbol Device:C
- added C14, C15, C16: 22uF, symbol Device:C
- added C6, C7: 0.1uF, symbol Device:C
- added C8: 10uF, symbol Device:C
- added C9: 2.2uF, symbol Device:C
- added L1: 1.2uH, symbol Device:L
- added R10, R11: 100K, symbol Device:R_US
- added R12: 56K, symbol Device:R_US
- added R13: 360k, symbol Device:R_US
- added R9: 255K, symbol Device:R_US
Connections:
- net at U5.1 (VCC): now also C9.2
- net at U5.10 (SS): now also C10.2
- net VOUT_call: now reaches U5.14 (VOUT)
- net VOUT_call: now also U5.15 (VOUT), U5.16 (VOUT), C13.1, C14.1, C15.1, C16.1, R13.2
- net at U5.17 (FB): now also R12.1, R13.1
- net at U5.18 (COMP): now also C12.2, R11.2
- net at U5.19 (ILIM): now also R10.2
- net EN: now reaches U5.2 (EN)
- net GND: now reaches U5.20 (AGND)
- net GND: now also U5.21 (PGND), C10.1, C11.1, C12.1, C13.2, C14.2, C15.2, C16.2, C7.2, C8.2, C9.1, R10.1, R12.2
- net at U5.3 (FSW): now also R9.1
- net at U5.4 (SW): now also U5.5 (SW), U5.6 (SW), U5.7 (SW), C6.2, L1.1, R9.2
- net at U5.8 (BOOT): now also C6.1
- net VIN: now reaches U5.9 (VIN)
- net VIN: now also C7.1, C8.1, L1.2
- new net: C11.2, R11.1

Commit message: update some things
Parts:
- R10, R11, R12, R13, R9: footprint (none) -> Resistor_SMD:R_0603_1608Metric
- U5: footprint RHL0020A -> footprints:RHL0020A
Changed lines of the file:
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@@
 			)
 		)
-		(property "Footprint" ""
+		(property "Footprint" "Resistor_SMD:R_0603_1608Metric"
 			(at 235.204 105.664 90)
 			(effects
@@
 			)
 		)
-		(property "Footprint" ""
+		(property "Footprint" "Resistor_SMD:R_0603_1608Metric"
 			(at 112.014 95.504 90)
 			(effects
@@
 			)
 		)
-		(property "Footprint" ""
+		(property "Footprint" "Resistor_SMD:R_0603_1608Metric"
 			(at 108.204 87.884 90)
 			(effects
@@
 			)
 		)
-		(property "Footprint" ""
+		(property "Footprint" "Resistor_SMD:R_0603_1608Metric"
 			(at 221.234 98.806 90)
 			(effects
@@
 			)
 		)
-		(property "Footprint" ""
+		(property "Footprint" "Resistor_SMD:R_0603_1608Metric"
 			(at 169.164 85.344 90)
 			(effects
@@
 			)
 		)
-		(property "Footprint" "RHL0020A"
+		(property "Footprint" "footprints:RHL0020A"
 			(at 146.05 91.44 0)
 			(effects

Commit message: add one batt
add one bat
Parts:
- removed C10, C11, C12: 47nF, symbol Device:C
- removed C13: 1uF, symbol Device:C
- removed C14, C15, C16: 22uF, symbol Device:C
- removed C6, C7: 0.1uF, symbol Device:C
- removed C8: 10uF, symbol Device:C
- removed C9: 2.2uF, symbol Device:C
- removed L1: 1.2uH, symbol Device:L
- removed R10, R11: 100K, Resistor_SMD:R_0603_1608Metric, symbol Device:R_US
- removed R12: 56K, Resistor_SMD:R_0603_1608Metric, symbol Device:R_US
- removed R13: 360k, Resistor_SMD:R_0603_1608Metric, symbol Device:R_US
- removed R9: 255K, Resistor_SMD:R_0603_1608Metric, symbol Device:R_US
- removed U5: TPS61088RHLR, footprints:RHL0020A, symbol TPS61088RHLR:TPS61088RHLR
Other:
- title: (none) -> Change to one cell

Commit message: push
Parts:
- added C11: 10uC, symbol Device:C
- added C6: 10uF, symbol Device:C
- added C8: 100nF, symbol Device:C
- added D7, D8: LED, symbol Device:LED
- added Q3: FS8205A, SOT-23-6L_TCP, symbol FS8205A:FS8205A
- added R10: 1K, Resistor_SMD:R_0402_1005Metric, symbol Device:R_US
- added R11: 1.5K, Resistor_SMD:R_0402_1005Metric, symbol Device:R_US
- added R15: 1K, symbol Device:R_US
- added R16: 100, symbol Device:R_US
- added R9: 1, Resistor_SMD:R_0402_1005Metric, symbol Device:R_US
- added U5: TP4056, Package_SO:MSOP-8-1EP_3x3mm_P0.65mm_EP1.5x1.8mm, symbol ul_TP4056:TP4056
- added U6: DW01A, Package_TO_SOT_SMD:SOT-23-6, symbol Battery_Management:DW01A
Connections:
- new net: C6.1, R9.2
- new net: Q3.4, U6.1 (OD)
- new net: R15.2, U6.2 (CS)
- new net: Q3.6, U6.3 (OC)
- new net: C8.1, R16.2, U6.5 (VCC)
- new net: R11.1, U5.2 (PROG)
- new net: D8.1 (K), U5.6 (*STDBY)
- new net: D7.1 (K), U5.7 (*CHRG)
- new net: D7.2 (A), D8.2 (A), R10.2
- new net +5V: R10.1, R9.1, U5.4 (VCC), U5.8 (CE)
- new net 4.2V: C11.1, R16.1, U5.5 (BAT)
- new net BAT-: C8.2, Q3.3, U6.6 (GND)
- new net GND: C11.2, C6.2, Q3.1, R11.2, R15.1, U5.1 (TEMP), U5.3 (GND)
- no-connect marks 0 -> 1

Commit message: ADD REV
DADA
Parts:
- added BZ1: Buzzer, symbol Device:Buzzer
- added Q4: Q_NPN_BEC, symbol Device:Q_NPN_BEC
- added R27, R28, R29: 1K, symbol Device:R_US
Connections:
- net GND: now also U5.EPAD, Q4.2 (E), R28.2
- new net: Q4.1 (B), R28.1, R29.1
- new net: BZ1.2 (-), Q4.3 (C), R27.2
- new net +3V3: BZ1.1 (+), R27.1
- new net BUZZER: R29.2

Commit message: adad
dada
Parts:
- removed D7, D8: LED, symbol Device:LED
- added D6, D7: SS14, Diode_SMD:D_SMA, symbol Diode:SS14
- BZ1: footprint (none) -> Buzzer_Beeper:Buzzer_15x7.5RM7.6
- C11, C6, C8: footprint (none) -> Capacitor_SMD:C_0603_1608Metric
- Q3: footprint SOT-23-6L_TCP -> footprints:SOT-23-6L_TCP
- R15, R16, R27, R28, R29: footprint (none) -> Resistor_SMD:R_0402_1005Metric
Connections:
- net at U5.6 (*STDBY): now also D6.1 (K)
- net at U5.7 (*CHRG): now also D7.1 (K)
- net at R10.2: now also D6.2 (A), D7.2 (A)
Other:
- moved on the sheet: R10, R9
