File: pg_hw/LCD.kicad_sch (KiCad schematic)
At the start: 1 part, among them J4 ILI1934

Commit message: push
Parts:
- added C12, C13, C14, C15, C16, C17, C18, C19, C20, C7: C, symbol Device:C
- added R17, R18, R19, R20, R21, R22, R23, R24, R25, R26: R, symbol Device:R
- added TP1, TP2, TP3, TP4, TP5: TestPoint_Flag, symbol Connector:TestPoint_Flag
- added U10, U11, U12, U8, U9: ~, symbol TTP:ttp233
Connections:
- net +3V3: now also C12.1, C14.1, C16.1, C18.1, C20.1, R17.2, R18.2, R19.2, R20.2, R21.2, R22.2, R23.2, R24.2, R25.2, R26.2, U10.5 (VDD), U11.5 (VDD), U12.5 (VDD), U8.5 (VDD), U9.5 (VDD)
- net GND: now also C12.2, C13.2, C14.2, C15.2, C16.2, C17.2, C18.2, C19.2, C20.2, C7.2, U10.2 (VSS), U11.2 (VSS), U12.2 (VSS), U8.2 (VSS), U9.2 (VSS)
- new net: R18.1, U8.6 (TOG)
- new net: C15.1, TP3.1, U10.3 (I)
- new net: R22.1, U10.4 (AHLB)
- new net: R21.1, U10.6 (TOG)
- new net: C13.1, TP2.1, U9.3 (I)
- new net: R20.1, U9.4 (AHLB)
- new net: R19.1, U9.6 (TOG)
- new net: C7.1, TP1.1, U8.3 (I)
- new net: R17.1, U8.4 (AHLB)
- new net: R23.1, U11.6 (TOG)
- new net: C19.1, TP5.1, U12.3 (I)
- new net: C17.1, TP4.1, U11.3 (I)
- new net: R24.1, U11.4 (AHLB)
- new net: R25.1, U12.6 (TOG)
- new net: R26.1, U12.4 (AHLB)
- new net Q_touch_1: U8.1 (Q)
- new net Q_touch_2: U9.1 (Q)
- new net Q_touch_3: U10.1 (Q)
- new net Q_touch_4: U11.1 (Q)
- new net Q_touch_5: U12.1 (Q)
Other:
- moved on the sheet: J4

Commit message: ADD REV
DADA
Connections:
- net DC renamed LCD_DC
- net LED renamed LED_LCD
- net RESET renamed LCD_RESET
Other:
- moved on the sheet: C12, C13

Commit message: Mungkin masih akan ada refisi
munvkin
Parts:
- added J2: Conn_01x06_Pin, symbol Connector:Conn_01x06_Pin
Connections:
- net +3V3: now also J2.6 (Pin_6)
- net GND: now also J2.5 (Pin_5)
- new net CTP_INT: J2.2 (Pin_2)
- new net CTP_RST: J2.1 (Pin_1)
- new net CTP_SCL: J2.4 (Pin_4)
- new net CTP_SDA: J2.3 (Pin_3)

Commit message: charlotte andeh
charlotte andeh
Parts:
- removed J4: ILI1934, symbol Connector:Conn_01x14_Pin
- added J3: Conn_01x40, symbol Connector_Generic:Conn_01x40
Connections:
- net +3V3: now also J3.7 (Pin_7)
- net GND: now also J3.16 (Pin_16), J3.5 (Pin_5)
- net LCD_DC: now also J3.10 (Pin_10)
- net LCD_RESET: now also J3.15 (Pin_15)
- net LED_LCD: now also J3.33 (Pin_33)
- net SPI1_CS: now also J3.9 (Pin_9)
- net SPI1_MISO: now also J3.14 (Pin_14)
- net SPI1_MOSI: now also J3.13 (Pin_13)

Commit message: addd draw
Changed lines of the file:
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@@
+	(wire
+		(pts
+			(xy 104.14 176.53) (xy 104.14 144.78)
+		)
+		(stroke
+			(width 0)
+			(type default)
+		)
+	)
 	(wire
 		(pts
@@
 		(pts
 			(xy 170.18 116.84) (xy 170.18 120.65)
-		)
-		(stroke
-			(width 0)
-			(type default)
-		)
-	)
-	(wire
-		(pts
-			(xy 71.12 86.36) (xy 39.37 86.36)
 		)
 		(stroke
@@
 		)
 	)
+	(label "SCK"
+		(at 104.14 165.1 270)
+		(fields_autoplaced yes)
+		(effects
+			(font
+				(size 1.27 1.27)
+			)
+			(justify right bottom)
+		)
+	)
 	(label "GND"
 		(at 120.65 167.64 270)
@@
 			)
 			(justify right bottom)
-		)
-	)
-	(label "SCK"
-		(at 59.69 86.36 0)
-		(fields_autoplaced yes)
-		(effects
-			(font
-				(size 1.27 1.27)
-			)
-			(justify left bottom)
 		)
 	)
@@
 		)
 	)
+	(global_label "SPI1_CLK"
+		(shape input)
+		(at 104.14 144.78 90)
+		(fields_autoplaced yes)
+		(effects
+			(font
+				(size 1.27 1.27)
+			)
+			(justify left)
+		)
+		(property "Intersheetrefs" "${INTERSHEET_REFS}"
+			(at 104.14 132.9653 90)
+			(effects
+				(font
+					(size 1.27 1.27)
+				)
+				(justify left)
+				(hide yes)
+			)
+		)
+	)
 	(global_label "SPI1_MISO"
 		(shape input)
@@
 			(effects
 				(font
-					(size 1.27 1.27)
-				)
-				(justify right)
-				(hide yes)
-			)
-		)
-	)
-	(global_label "SPI1_CLK"
-		(shape input)
-		(at 39.37 86.36 180)
-		(fields_autoplaced yes)
-		(effects
-			(font
-				(size 1.27 1.27)
-			)
-			(justify right)
-		)
-		(property "Intersheetrefs" "${INTERSHEET_REFS}"
-			(at 27.5553 86.36 0)
-			(effects
-				(font

Commit message: update ke lcd
lcd diupdate
Parts:
- added R36: 1k, symbol Device:R
- added R37: 0, symbol Device:R
Connections:
- net +3V3: now also R36.1, R37.1
- net GND: now also J3.38 (Pin_38)
- net LCD_DC: now also J3.11 (Pin_11); no longer J3.10 (Pin_10)
- net SPI1_CLK: now also J3.10 (Pin_10)
- net at J3.39 (Pin_39): now also J3.40 (Pin_40), R36.2, R37.2

Commit message: usb revision
add some revision
Parts:
- removed C19, C20: C, symbol Device:C
- removed R25, R26: R, symbol Device:R
- removed TP5: TestPoint_Flag, symbol Connector:TestPoint_Flag
- removed U12: ~, symbol TTP:ttp233
- J2: value Conn_01x06_Pin -> FPC_Touch
- J3: value Conn_01x40 -> FPC_Display
- U10, U11, U8: value ~ -> ttp233
- U9: value ~ -> TTP233

Commit message: adad
dada
Parts:
- C12, C13, C14, C15, C16, C17, C18, C7: footprint (none) -> Capacitor_SMD:C_0603_1608Metric
- R17, R18, R19, R20, R21, R22, R23, R24, R36, R37: footprint (none) -> Resistor_SMD:R_0402_1005Metric
Other:
- moved on the sheet: C12, C13, C14, C15, C16, C17, C18, C7, R17, R18, R19, R20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
