File: pg_hw/BMS.kicad_sch (KiCad schematic)
At the start: 3 parts, among them U4 BQ25703ARSNT

Commit message: updarte schematics
schematics menuju pengecheckan
Parts:
- added C17: 0.047uF, symbol Device:C
- added C18, C19: 150pF, symbol Device:C
- added C20, C21, C22, C23, C24, C28, C43, C44, C45, C46, C47, C48: 10uF, symbol Device:C
- added C25: 47uF, symbol Device:C_Polarized_US
- added C26, C39, C50: 1uF, symbol Device:C
- added C27, C49, C51, C52: 0.1uF, symbol Device:C
- added C29: 2.2uF, symbol Device:C
- added C30: 15pF, symbol Device:C
- added C31: 680pF, symbol Device:C
- added C32, C33, C40: 100pF, symbol Device:C
- added C34: 1nF, symbol Device:C
- added C35: 0.01uF, symbol Device:C
- added C36: 0.47uF, symbol Device:C
- added C37, C38: 0.033uF, symbol Device:C
- added C41: 1800pF, symbol Device:C
- added C42: 33pF, symbol Device:C
- added D10, D11: D_Zener, symbol Device:D_Zener
- added D7: 30V, symbol Device:D_Zener
- added D8: SMAJ26CA, Diode_SMD:D_SMA, symbol Diode:SMAJ26CA
- added D9: LED, symbol Device:LED
- added J10, J14, J15, J16, J5, J6, J7, J9: Conn_01x02_Pin, symbol Connector:Conn_01x02_Pin
- added J11, J12: Conn_01x04_Pin, symbol Connector:Conn_01x04_Pin
- added J13, J8: Conn_01x03_Pin, symbol Connector:Conn_01x03_Pin
- added L2: 2.2uH, symbol Device:L_Ferrite
- added Q3, Q4, Q5, Q6: CSD17551Q3A, CSD17551Q3A:TRANS_CSD18543Q3A, symbol CSD17551Q3A:CSD17551Q3A
- added Q7, Q8: DMP3035SFG-7, POWERDI3333-8_3P3X3P3_DIO, symbol DMP3035SFG_7:DMP3035SFG-7
- added Q9: DCX124EK-7-F, SOT26-DCX124_DIO, symbol DCX124EK_7_F:DCX124EK-7-F
- added R14, R16, R43, R48: 10, symbol Device:R_US
- added R15, R27: 0.01, symbol Device:R_US
- added R17, R39, R44: 10K, symbol Device:R_US
- added R18, R23, R38: 300k, symbol Device:R_US
- added R19, R42: 100k, symbol Device:R_US
- added R20: 280K, symbol Device:R_US
- added R21: 120K, symbol Device:R_US
- added R22: 64.9k, symbol Device:R_US
- added R24: NET_TIE, symbol Device:R
- added R25: 137k, symbol Device:R_US
- added R26, R28: 4.99, symbol Device:R_US
- added R29: 10.0, symbol Device:R_US
- added R30: 383k, symbol Device:R_US
- added R31: 220K, symbol Device:R_US
- added R32: 383K, symbol Device:R_US
- added R33: 40.2k, symbol Device:R_US
- added R34: 10k, symbol Device:R_US
- added R35: 100, symbol Device:R_US
- added R36: 100K, symbol Device:R_US
- added R37: 2.0M, symbol Device:R_US
- added R40: 1.0, symbol Device:R_US
- added R41: 20k, symbol Device:R_US
- added R45, R46: 3.9, symbol Device:R_US
- added R47: 2.00k, symbol Device:R_US
- added TP1: HIDRV1, symbol Connector:TestPoint
- added TP2: LODRV1, symbol Connector:TestPoint
- added TP3, TP4: BTST1, symbol Connector:TestPoint
- added TP5: VSYS, symbol Connector:TestPoint
- added TP6: PROCHOT, symbol Connector:TestPoint
- added TP7: TestPoint, symbol Connector:TestPoint
- added U10: LM3480IM3-3.3/NOPB, DBZ0003A_N, symbol LM3480IM3_3_3_NOPB:LM3480IM3-3.3_NOPB
- added U6: CSD25402Q3A, CSD25402Q3A, symbol CSD25402Q3A:CSD25402Q3A
- added U7, U8, U9: 2N7002ET1G, SOT-23_ONS, symbol 2N7002ET1G:2N7002ET1G
- R7, R8: value 4.7K -> 10K
Connections:
- net +3V3: now also R32.2, R34.2, R35.2, R36.2, R39.2, R44.2, R47.1
- net GND: now also C30.1, C31.1, C32.1, C33.1, C36.2, C37.2, C38.2, C39.2, C40.1, C41.1, C42.1, J10.1 (Pin_1), J11.1 (Pin_1), J13.2 (Pin_2), J5.1 (Pin_1), R18.2, R19.2, R23.2, R24.2, R25.2, R31.1, R38.2, U7.2 (S), U8.2 (S), U9.2 (S); no longer U4.27 (PGND), U4.33 (PAD)
- net SCL_BMS: now also J11.2 (Pin_2)
- net SDA_BMS: now also J11.3 (Pin_3)
- net VBUS: now reaches U4.1 (VBUS)
- net VBUS: now also C36.1, D11.2 (A), J8.2 (Pin_2)
- net at U4.10 (PSYS): now also R23.1
- net at U4.11 (PROCHOT_N): now also R34.1, TP6.1
- net at U4.14 (CMPIN): now also J13.3 (Pin_3), R37.1, R38.1
- net at U4.15 (CMPOUT): now also J13.1 (Pin_1), R37.2, R39.1
- net at U4.16 (COMP1): now also C42.2, R33.1
- net at U4.17 (COMP2): now also C30.2, R17.1
- net at U4.18 (CELL_BATPRES): now also J5.2 (Pin_2), J6.2 (Pin_2), J7.1 (Pin_1), R19.1, R20.2, U7.3 (D)
- net at U4.19 (SRN): now also R16.2
- net at U4.2 (ACN): now also C37.1, R26.2
- net at U4.20 (SRP): now also R14.2
- net at U4.21 (BATDRV_N): now also U6.4 (G)
- net at U4.22 (VSYS): now also C20.2, C21.2, C22.2, C23.2, C24.2, C25.1, Q5.10 (D__5), Q5.11 (D__6), Q5.12 (D__7), Q5.5 (D), Q5.6 (D__1), Q5.7 (D__2), Q5.8 (D__3), Q5.9 (D__4), TP5.1, U6.5 (S), U6.6 (S), U6.7 (S), U6.8 (S), U6.9 (S)
- net at U4.23 (SW2): now also U4.25 (BTST2), L2.2, Q5.1 (S), Q5.2 (S__1), Q5.3 (S__2), Q6.10 (D__5), Q6.11 (D__6), Q6.12 (D__7), Q6.5 (D), Q6.6 (D__1), Q6.7 (D__2), Q6.8 (D__3), Q6.9 (D__4)
- net at U4.24 (HIDRV2): now also Q5.4 (G)
- net at U4.26 (LODRV2): now also C19.1, Q6.4 (G)
- net at U4.28 (REGN): now also C29.2
- net at U4.29 (LODRV1): now also C18.1, Q4.4 (G), TP2.1
- net at U4.3 (ACP): now also C38.1, R28.2
- net at U4.30 (BTST1): now also C17.2, TP3.1
- net at U4.31 (HIDRV1): now also Q3.4 (G), TP1.1
- net at U4.32 (SW1): now also C17.1, L2.1, Q3.1 (S), Q3.2 (S__1), Q3.3 (S__2), Q4.10 (D__5), Q4.11 (D__6), Q4.12 (D__7), Q4.5 (D), Q4.6 (D__1), Q4.7 (D__2), Q4.8 (D__3), Q4.9 (D__4), TP4.1
- net CHG_OK: now reaches U4.4 (CHRG_OK)
- net CHG_OK: now also J12.2 (Pin_2), R36.1, U8.1 (G), U9.1 (G)
- net at U4.5 (EN_OTG): now also J12.3 (Pin_3)
- net ILIM_HIZ: now reaches U4.6 (ILIM_HIZ)
- net ILIM_HIZ: now also C40.2, D7.2 (A), R30.2, R31.2
- net VDDA: now reaches U4.7 (VDDA)
- net VDDA: now also C39.1, J9.2 (Pin_2), R21.1, R22.1, R29.2
- net at U4.8 (IADPT): now also C33.2, R25.1
- net at U4.9 (IBAT): now also C32.2
- new net: C26.2, C27.2, R14.1, R15.1, U6.1 (D), U6.2 (D), U6.3 (D)
- new net: C50.1, R45.1, R46.1
- new net: C43.1, C44.1, C45.1, C46.1, C47.1, C48.1, J16.1 (Pin_1), Q7.5, Q7.6, Q7.7, Q7.8, R27.1, R28.1
- new net: C34.1, C35.1, J8.1 (Pin_1), Q3.10 (D__5), Q3.11 (D__6), Q3.12 (D__7), Q3.5 (D), Q3.6 (D__1), Q3.7 (D__2), Q3.8 (D__3), Q3.9 (D__4), R26.1, R27.2
- new net: C31.2, R17.2
- new net: J6.1 (Pin_1), R20.1, R21.2
- new net: J9.1 (Pin_1), R30.1
- new net: C49.1, D8.2 (A2), Q7.1, Q7.2, Q7.3, Q8.1, Q8.2, Q8.3, R42.2, R43.2
- new net: C49.2, Q7.4, Q8.4, Q9.4, R41.2, R42.1
- new net: C51.1, J15.2 (Pin_2), U10.2 (IN)
- new net: C41.2, R33.2
- new net: Q9.1, Q9.5
- new net: Q9.2, R44.1, U9.3 (D)
- new net: Q9.3, R43.1
- new net: D10.1 (K), D11.1 (K), R48.1
- new net: J7.2 (Pin_2), R22.2
- new net: J15.1 (Pin_1), R48.2
- new net: J11.4 (Pin_4), R35.1
- new net: D9.1 (K), U8.3 (D)
- new net: D9.2 (A), R47.2
- new net: J8.3 (Pin_3), R40.2
- new net 3V3: C52.1, U10.1 (OUT)
- new net BAT: C27.1, C28.2, D10.2 (A), R15.2, R16.1
- new net CELL_control: J12.4 (Pin_4), R18.1, U7.1 (G)
- new net GNDPWR: C18.2, C19.2, C20.1, C21.1, C22.1, C23.1, C24.1, C25.2, C26.1, C28.1, C29.1, C34.2, C35.2, C43.2, C44.2, C45.2, C46.2, C47.2, C48.2, C50.2, C51.2, C52.2, D8.1 (A1), J14.2 (Pin_2), Q4.1 (S), Q4.2 (S__1), Q4.3 (S__2), Q6.1 (S), Q6.2 (S__1), Q6.3 (S__2), Q9.6, R24.1, R41.1, U10.3 (GND), U4.27 (PGND), U4.33 (PAD)
- new net ILIM_control: D7.1 (K), J10.2 (Pin_2), J12.1 (Pin_1), R32.1
- new net REGN: R29.1
- new net VIN: J14.1 (Pin_1), J16.2 (Pin_2), Q8.5, Q8.6, Q8.7, Q8.8, R40.1, R45.2, R46.2, TP7.1
Other:
- moved on the sheet: R7, R8, U4

Commit message: update some things
Parts:
- J10, J14, J15, J16, J5, J6, J7, J9: footprint (none) -> Connector_PinHeader_2.54mm:PinHeader_1x02_P2.54mm_Vertical
- J11, J12: footprint (none) -> Connector_PinHeader_2.54mm:PinHeader_1x04_P2.54mm_Vertical
- J13, J8: footprint (none) -> Connector_PinHeader_2.54mm:PinHeader_1x03_P2.54mm_Vertical
- Q3, Q4, Q5, Q6: footprint CSD17551Q3A:TRANS_CSD18543Q3A -> footprints:DNH0008A
- Q7, Q8: footprint POWERDI3333-8_3P3X3P3_DIO -> footprints:POWERDI3333-8_3P3X3P3_DIO
- Q9: footprint SOT26-DCX124_DIO -> footprints:SOT26-DCX124_DIO
- R14, R15, R16, R17, R18, R19, R20, R21, R22, R23, R24, R25, R26, R27, R28, R29, R30, R31, R32, R33, R34, R35, R36, R37, R38, R39, R40, R41, R42, R43, R44, R45, R46, R47, R48, R7, R8: footprint (none) -> Resistor_SMD:R_0603_1608Metric
- TP7: footprint (none) -> TestPoint:TestPoint_2Pads_Pitch2.54mm_Drill0.8mm
- U10: footprint DBZ0003A_N -> footprints:DBZ0003A_N
- U4: footprint RSN0032B -> footprints:RSN0032B
- U6: footprint CSD25402Q3A -> footprints:CSD25402Q3A
- U7, U8, U9: footprint SOT-23_ONS -> footprints:SOT-23_ONS
Changed lines of the file:
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@@
 			)
 		)
-		(property "Footprint" "CSD25402Q3A"
+		(property "Footprint" "footprints:CSD25402Q3A"
 			(at 452.12 162.56 0)
 			(effects
@@
 			)
 		)
-		(property "Footprint" ""
+		(property "Footprint" "Resistor_SMD:R_0603_1608Metric"
 			(at 48.514 139.446 90)
 			(effects
@@
 			)
 		)
-		(property "Footprint" ""
+		(property "Footprint" "Resistor_SMD:R_0603_1608Metric"
 			(at 275.336 290.576 90)
 			(effects
@@
 			)
 		)
-		(property "Footprint" ""
+		(property "Footprint" "Resistor_SMD:R_0603_1608Metric"
 			(at 344.424 211.074 90)
 			(effects
@@
 			)
 		)
-		(property "Footprint" ""
+		(property "Footprint" "Connector_PinHeader_2.54mm:PinHeader_1x02_P2.54mm_Vertical"
 			(at 210.82 220.98 0)
 			(effects
@@
 			)
 		)
-		(property "Footprint" ""
+		(property "Footprint" "Resistor_SMD:R_0603_1608Metric"
 			(at 385.826 241.554 90)
 			(effects
@@
 			)
 		)
-		(property "Footprint" ""
+		(property "Footprint" "Connector_PinHeader_2.54mm:PinHeader_1x02_P2.54mm_Vertical"
 			(at 97.79 102.87 0)
 			(effects
@@
 			)
 		)
-		(property "Footprint" ""
+		(property "Footprint" "Resistor_SMD:R_0603_1608Metric"
 			(at 475.234 164.084 90)
 			(effects
@@
 			)
 		)
-		(property "Footprint" ""
+		(property "Footprint" "Resistor_SMD:R_0603_1608Metric"
 			(at 462.026 235.966 90)
 			(effects
@@
 			)
 		)
-		(property "Footprint" ""
+		(property "Footprint" "Resistor_SMD:R_0603_1608Metric"
 			(at 38.354 139.446 90)
 			(effects
@@
 			)
 		)
-		(property "Footprint" ""
+		(property "Footprint" "Resistor_SMD:R_0603_1608Metric"
 			(at 242.316 206.756 90)
 			(effects
@@
 			)
 		)
-		(property "Footprint" "POWERDI3333-8_3P3X3P3_DIO"
+		(property "Footprint" "footprints:POWERDI3333-8_3P3X3P3_DIO"
 			(at 86.36 133.35 0)
 			(effects
@@
 			)
 		)
-		(property "Footprint" "CSD17551Q3A:TRANS_CSD18543Q3A"
+		(property "Footprint" "footprints:DNH0008A"
 			(at 260.35 121.92 0)
 			(effects
@@
 			)
 		)
-		(property "Footprint" "SOT-23_ONS"
+		(property "Footprint" "footprints:SOT-23_ONS"
 			(at 401.32 248.92 0)
 			(effects
@@
 			)
 		)
-		(property "Footprint" ""
+		(property "Footprint" "Resistor_SMD:R_0603_1608Metric"
 			(at 349.25 258.318 90)
 			(effects
@@
 			)
 		)
-		(property "Footprint" ""
+		(property "Footprint" "Connector_PinHeader_2.54mm:PinHeader_1x02_P2.54mm_Vertical"
 			(at 19.05 137.16 0)
 			(effects
@@
 			)
 		)
-		(property "Footprint" "DBZ0003A_N"
+		(property "Footprint" "footprints:DBZ0003A_N"
 			(at 393.7 344.17 0)
 			(effects
@@
 			)
 		)
-		(property "Footprint" ""
+		(property "Footprint" "Resistor_SMD:R_0603_1608Metric"
 			(at 230.124 218.186 90)
 			(effects
@@
 			)
 		)
-		(property "Footprint" "CSD17551Q3A:TRANS_CSD18543Q3A"
+		(property "Footprint" "footprints:DNH0008A"
 			(at 331.47 110.49 0)
 			(effects
@@
 			)
 		)
-		(property "Footprint" "SOT26-DCX124_DIO"
+		(property "Footprint" "footprints:SOT26-DCX124_DIO"
 			(at 67.31 185.42 0)
 			(effects
@@
 			)
 		)
-		(property "Footprint" ""
+		(property "Footprint" "Resistor_SMD:R_0603_1608Metric"
 			(at 281.686 213.106 90)
 			(effects
@@
 			)
 		)
-		(property "Footprint" ""
+		(property "Footprint" "Resistor_SMD:R_0603_1608Metric"
 			(at 106.934 164.846 90)
 			(effects
@@
 			)
 		)
-		(property "Footprint" ""
+		(property "Footprint" "Resistor_SMD:R_0603_1608Metric"
 			(at 175.514 136.144 90)
 			(effects
@@
 			)
 		)
-		(property "Footprint" ""
+		(property "Footprint" "Connector_PinHeader_2.54mm:PinHeader_1x02_P2.54mm_Vertical"
 			(at 471.17 245.11 0)
 			(effects
@@
 			)
 		)
-		(property "Footprint" ""
+		(property "Footprint" "Connector_PinHeader_2.54mm:PinHeader_1x02_P2.54mm_Vertical"
 			(at 320.04 372.11 0)
 			(effects
@@
 			)
 		)
-		(property "Footprint" ""
+		(property "Footprint" "Resistor_SMD:R_0603_1608Metric"
 			(at 355.346 245.364 90)
 			(effects
@@
 			)
 		)
-		(property "Footprint" ""
+		(property "Footprint" "Resistor_SMD:R_0603_1608Metric"
 			(at 178.054 211.836 90)
 			(effects
@@
 			)
 		)
-		(property "Footprint" "SOT-23_ONS"
+		(property "Footprint" "footprints:SOT-23_ONS"
 			(at 78.74 213.36 0)
 			(effects
@@
 			)
 		)
-		(property "Footprint" ""
+		(property "Footprint" "Resistor_SMD:R_0603_1608Metric"
 			(at 166.624 251.206 90)
 			(effects
@@
 			)
 		)
-		(property "Footprint" ""
+		(property "Footprint" "Resistor_SMD:R_0603_1608Metric"
 			(at 230.124 193.294 90)
 			(effects
@@
 			)
 		)
-		(property "Footprint" ""
+		(property "Footprint" "Connector_PinHeader_2.54mm:PinHeader_1x02_P2.54mm_Vertical"
 			(at 254 205.74 0)
 			(effects
@@
 			)
 		)
-		(property "Footprint" ""
+		(property "Footprint" "Resistor_SMD:R_0603_1608Metric"
 			(at 199.644 276.606 90)
 			(effects
@@
 			)
 		)
-		(property "Footprint" "RSN0032B"
+		(property "Footprint" "footprints:RSN0032B"
 			(at 314.96 204.47 0)
 			(effects
@@
 			)
 		)
-		(property "Footprint" ""
+		(property "Footprint" "Resistor_SMD:R_0603_1608Metric"
 			(at 276.606 313.944 90)
 			(effects
@@
 			)
 		)
-		(property "Footprint" ""
+		(property "Footprint" "Resistor_SMD:R_0603_1608Metric"
 			(at 479.806 235.966 90)
 			(effects
@@
 			)
 		)
-		(property "Footprint" ""
+		(property "Footprint" "Resistor_SMD:R_0603_1608Metric"
 			(at 183.896 145.034 90)
 			(effects
@@
 			)
 		)
-		(property "Footprint" ""
+		(property "Footprint" "Resistor_SMD:R_0603_1608Metric"
 			(at 319.786 349.504 90)
 			(effects
@@
 			)
 		)
-		(property "Footprint" ""
+		(property "Footprint" "Resistor_SMD:R_0603_1608Metric"
 			(at 453.136 252.984 90)
 			(effects
@@
 			)
 		)
-		(property "Footprint" "CSD17551Q3A:TRANS_CSD18543Q3A"
+		(property "Footprint" "footprints:DNH0008A"
 			(at 212.09 119.38 0)
 			(effects
@@
 			)
 		)
-		(property "Footprint" ""
+		(property "Footprint" "Resistor_SMD:R_0603_1608Metric"
 			(at 275.336 218.186 90)
 			(effects
@@
 			)
 		)
-		(property "Footprint" "SOT-23_ONS"
+		(property "Footprint" "footprints:SOT-23_ONS"
 			(at 160.02 367.03 0)
 			(effects
@@
 			)
 		)
-		(property "Footprint" "CSD17551Q3A:TRANS_CSD18543Q3A"
+		(property "Footprint" "footprints:DNH0008A"
 			(at 403.86 110.49 0)
 			(effects
@@
 			)
 		)
-		(property "Footprint" ""
+		(property "Footprint" "Resistor_SMD:R_0603_1608Metric"
 			(at 76.454 155.956 90)
 			(effects
@@
 			)
 		)
-		(property "Footprint" ""
+		(property "Footprint" "Connector_PinHeader_2.54mm:PinHeader_1x04_P2.54mm_Vertical"
 			(at 156.21 262.89 0)
 			(effects
@@
 			)
 		)
-		(property "Footprint" ""
+		(property "Footprint" "Connector_PinHeader_2.54mm:PinHeader_1x02_P2.54mm_Vertical"
 			(at 463.55 217.17 0)
 			(effects
@@
 			)
 		)
-		(property "Footprint" ""
+		(property "Footprint" "Resistor_SMD:R_0603_1608Metric"
 			(at 483.616 181.864 90)
 			(effects
@@
 			)
 		)
-		(property "Footprint" ""
+		(property "Footprint" "Resistor_SMD:R_0603_1608Metric"
 			(at 239.014 219.456 90)
 			(effects
@@
 			)
 		)
-		(property "Footprint" ""
+		(property "Footprint" "Resistor_SMD:R_0603_1608Metric"
 			(at 200.914 210.566 90)
 			(effects
@@
 			)
 		)
-		(property "Footprint" ""
+		(property "Footprint" "Resistor_SMD:R_0603_1608Metric"
 			(at 203.454 155.956 90)
 			(effects
@@
 			)
 		)
-		(property "Footprint" ""
+		(property "Footprint" "Connector_PinHeader_2.54mm:PinHeader_1x02_P2.54mm_Vertical"
 			(at 478.79 251.46 0)
 			(effects
@@
 			)
 		)
-		(property "Footprint" ""
+		(property "Footprint" "Connector_PinHeader_2.54mm:PinHeader_1x04_P2.54mm_Vertical"
 			(at 156.21 283.21 0)
 			(effects
@@
 			)
 		)
-		(property "Footprint" ""
+		(property "Footprint" "Connector_PinHeader_2.54mm:PinHeader_1x03_P2.54mm_Vertical"
 			(at 207.01 307.34 0)
 			(effects
@@
 			)
 		)
-		(property "Footprint" ""
+		(property "Footprint" "Resistor_SMD:R_0603_1608Metric"
 			(at 95.504 153.416 90)
 			(effects
@@
 			)
 		)
-		(property "Footprint" ""
+		(property "Footprint" "Resistor_SMD:R_0603_1608Metric"
 			(at 479.806 241.046 90)
 			(effects
@@
 			)
 		)
-		(property "Footprint" ""
+		(property "Footprint" "Resistor_SMD:R_0603_1608Metric"
 			(at 171.196 145.034 90)
 			(effects
@@
 			)
 		)
-		(property "Footprint" ""
+		(property "Footprint" "Resistor_SMD:R_0603_1608Metric"
 			(at 397.256 256.794 90)
 			(effects
@@
 			)
 		)
-		(property "Footprint" ""
+		(property "Footprint" "Resistor_SMD:R_0603_1608Metric"
 			(at 470.916 181.864 90)
 			(effects
@@
 			)
 		)
-		(property "Footprint" "POWERDI3333-8_3P3X3P3_DIO"
+		(property "Footprint" "footprints:POWERDI3333-8_3P3X3P3_DIO"
 			(at 107.95 133.35 0)
 			(effects
@@
 			)
 		)
-		(property "Footprint" ""
+		(property "Footprint" "Connector_PinHeader_2.54mm:PinHeader_1x03_P2.54mm_Vertical"
 			(at 198.12 147.32 0)
 			(effects
@@
 			)
 		)
-		(property "Footprint" ""
+		(property "Footprint" "TestPoint:TestPoint_2Pads_Pitch2.54mm_Drill0.8mm"
 			(at 49.53 135.89 0)
 			(effects
@@
 			)
 		)
-		(property "Footprint" ""
+		(property "Footprint" "Resistor_SMD:R_0603_1608Metric"
 			(at 237.744 296.926 90)
 			(effects
@@
 			)
 		)
-		(property "Footprint" ""
+		(property "Footprint" "Resistor_SMD:R_0603_1608Metric"
 			(at 56.134 171.196 90)
 			(effects
@@
 			)
 		)
-		(property "Footprint" ""
+		(property "Footprint" "Resistor_SMD:R_0603_1608Metric"
 			(at 202.946 332.994 90)
 			(effects

Commit message: add one batt
add one bat
Parts:
- removed C17: 0.047uF, symbol Device:C
- removed C18, C19: 150pF, symbol Device:C
- removed C20, C21, C22, C23, C24, C28, C43, C44, C45, C46, C47, C48: 10uF, symbol Device:C
- removed C25: 47uF, symbol Device:C_Polarized_US
- removed C26, C39, C50: 1uF, symbol Device:C
- removed C27, C49, C51, C52: 0.1uF, symbol Device:C
- removed C29: 2.2uF, symbol Device:C
- removed C30: 15pF, symbol Device:C
- removed C31: 680pF, symbol Device:C
- removed C32, C33, C40: 100pF, symbol Device:C
- removed C34: 1nF, symbol Device:C
- removed C35: 0.01uF, symbol Device:C
- removed C36: 0.47uF, symbol Device:C
- removed C37, C38: 0.033uF, symbol Device:C
- removed C41: 1800pF, symbol Device:C
- removed C42: 33pF, symbol Device:C
- removed D10, D11: D_Zener, symbol Device:D_Zener
- removed D7: 30V, symbol Device:D_Zener
- removed D8: SMAJ26CA, Diode_SMD:D_SMA, symbol Diode:SMAJ26CA
- removed D9: LED, symbol Device:LED
- removed J10, J14, J15, J16, J5, J6, J7, J9: Conn_01x02_Pin, Connector_PinHeader_2.54mm:PinHeader_1x02_P2.54mm_Vertical, symbol Connector:Conn_01x02_Pin
- removed J11, J12: Conn_01x04_Pin, Connector_PinHeader_2.54mm:PinHeader_1x04_P2.54mm_Vertical, symbol Connector:Conn_01x04_Pin
- removed J13, J8: Conn_01x03_Pin, Connector_PinHeader_2.54mm:PinHeader_1x03_P2.54mm_Vertical, symbol Connector:Conn_01x03_Pin
- removed L2: 2.2uH, symbol Device:L_Ferrite
- removed Q3, Q4, Q5, Q6: CSD17551Q3A, footprints:DNH0008A, symbol CSD17551Q3A:CSD17551Q3A
- removed Q7, Q8: DMP3035SFG-7, footprints:POWERDI3333-8_3P3X3P3_DIO, symbol DMP3035SFG_7:DMP3035SFG-7
- removed Q9: DCX124EK-7-F, footprints:SOT26-DCX124_DIO, symbol DCX124EK_7_F:DCX124EK-7-F
- removed R14, R16, R43, R48: 10, Resistor_SMD:R_0603_1608Metric, symbol Device:R_US
- removed R15, R27: 0.01, Resistor_SMD:R_0603_1608Metric, symbol Device:R_US
- removed R17, R39, R44, R7, R8: 10K, Resistor_SMD:R_0603_1608Metric, symbol Device:R_US
- removed R18, R23, R38: 300k, Resistor_SMD:R_0603_1608Metric, symbol Device:R_US
- removed R19, R42: 100k, Resistor_SMD:R_0603_1608Metric, symbol Device:R_US
- removed R20: 280K, Resistor_SMD:R_0603_1608Metric, symbol Device:R_US
- removed R21: 120K, Resistor_SMD:R_0603_1608Metric, symbol Device:R_US
- removed R22: 64.9k, Resistor_SMD:R_0603_1608Metric, symbol Device:R_US
- removed R24: NET_TIE, Resistor_SMD:R_0603_1608Metric, symbol Device:R
- removed R25: 137k, Resistor_SMD:R_0603_1608Metric, symbol Device:R_US
- removed R26, R28: 4.99, Resistor_SMD:R_0603_1608Metric, symbol Device:R_US
- removed R29: 10.0, Resistor_SMD:R_0603_1608Metric, symbol Device:R_US
- removed R30: 383k, Resistor_SMD:R_0603_1608Metric, symbol Device:R_US
- removed R31: 220K, Resistor_SMD:R_0603_1608Metric, symbol Device:R_US
- removed R32: 383K, Resistor_SMD:R_0603_1608Metric, symbol Device:R_US
- removed R33: 40.2k, Resistor_SMD:R_0603_1608Metric, symbol Device:R_US
- removed R34: 10k, Resistor_SMD:R_0603_1608Metric, symbol Device:R_US
- removed R35: 100, Resistor_SMD:R_0603_1608Metric, symbol Device:R_US
- removed R36: 100K, Resistor_SMD:R_0603_1608Metric, symbol Device:R_US
- removed R37: 2.0M, Resistor_SMD:R_0603_1608Metric, symbol Device:R_US
- removed R40: 1.0, Resistor_SMD:R_0603_1608Metric, symbol Device:R_US
- removed R41: 20k, Resistor_SMD:R_0603_1608Metric, symbol Device:R_US
- removed R45, R46: 3.9, Resistor_SMD:R_0603_1608Metric, symbol Device:R_US
- removed R47: 2.00k, Resistor_SMD:R_0603_1608Metric, symbol Device:R_US
- removed TP1: HIDRV1, symbol Connector:TestPoint
- removed TP2: LODRV1, symbol Connector:TestPoint
- removed TP3, TP4: BTST1, symbol Connector:TestPoint
- removed TP5: VSYS, symbol Connector:TestPoint
- removed TP6: PROCHOT, symbol Connector:TestPoint
- removed TP7: TestPoint, TestPoint:TestPoint_2Pads_Pitch2.54mm_Drill0.8mm, symbol Connector:TestPoint
- removed U10: LM3480IM3-3.3/NOPB, footprints:DBZ0003A_N, symbol LM3480IM3_3_3_NOPB:LM3480IM3-3.3_NOPB
- removed U4: BQ25703ARSNT, footprints:RSN0032B, symbol BQ25703ARSNT:BQ25703ARSNT
- removed U6: CSD25402Q3A, footprints:CSD25402Q3A, symbol CSD25402Q3A:CSD25402Q3A
- removed U7, U8, U9: 2N7002ET1G, footprints:SOT-23_ONS, symbol 2N7002ET1G:2N7002ET1G
- added U4: TP4056, SOP8-PP_TPW, symbol ul_TP4056:TP4056
- added U5: MAX17048X+T10, 21-0555B_W80B1-1_MXM, symbol ul_MAX17048X-T10:MAX17048X+T10
Connections:
- net GND: now also U5.A4 (GND)
- net SCL_BMS: now also U5.B2 (SCL)
- net SDA_BMS: now also U5.B1 (SDA)

Commit message: change batt again
Parts:
- added C6: 10uF, symbol Device:C
- added C7: C, symbol Device:C
- added C8: 0.1uF, symbol Device:C_Polarized_US
- added D7, D8: LED, symbol Device:LED
- added R10: 1K, symbol Device:R_US
- added R11: RPROG, symbol Device:R_US
- added R12, R13: R_US, symbol Device:R_US
- added R9: 1, symbol Device:R_US
- U4: footprint SOP8-PP_TPW -> Package_SO:MSOP-8-1EP_3x3mm_P0.65mm_EP1.5x1.8mm
- U5: footprint 21-0555B_W80B1-1_MXM -> Package_SO:MSOP-8-1EP_3x3mm_P0.65mm_EP1.73x1.85mm
Connections:
- net GND: now also U4.3 (GND), U5.A1 (CTG), U5.B3 (QSTRT), C6.2, C7.2, C8.2, R11.2, R12.2
- net at U4.1 (TEMP): now also R12.1, R13.2
- net at U4.2 (PROG): now also R11.1
- net +5V: now reaches U4.4 (VCC)
- net +5V: now also U4.8 (CE), R10.1, R13.1, R9.1
- net at U4.5 (BAT): now also C7.1
- net at U4.6 (*STDBY): now also D7.1 (K)
- net at U4.7 (*CHRG): now also D8.1 (K)
- net BAT+: now reaches U5.A2 (CELL)
- net BAT+: now also U5.A3 (VDD), C8.1
- net INTERRUPT: now reaches U5.B4 (*ALRT)
- net SCL_BMS renamed LP_I2C_SCL
- net SDA_BMS renamed LP_I2C_SDA
- new net: C6.1, R9.2
- new net: D7.2 (A), D8.2 (A), R10.2
Other:
- moved on the sheet: U4, U5

Commit message: hui
Parts:
- removed C8: 0.1uF, symbol Device:C_Polarized_US
- removed U5: MAX17048X+T10, Package_SO:MSOP-8-1EP_3x3mm_P0.65mm_EP1.73x1.85mm, symbol ul_MAX17048X-T10:MAX17048X+T10
- added C10: 1uF, Capacitor_SMD:C_0603_1608Metric, symbol Device:C
- added C9: 0.47uF, Resistor_SMD:R_0603_1608Metric, symbol Device:C
- added R14: 0.01, Resistor_SMD:R_0402_1005Metric, symbol Device:R_US
- added U4: BQ27441DRZR-G1A, Copy of DRZ0012A, symbol BQ27441DRZR_G1A:BQ27441DRZR-G1A
- R10, R11, R12, R13, R9: footprint (none) -> Resistor_SMD:R_0402_1005Metric
Connections:
- net GND: now also C10.1, C10.2, C9.2, U4.3 (VSS), U4.6 (BAT)
- net LP_I2C_SCL: now also U4.2 (SCL)
- net LP_I2C_SDA: now also U4.1 (SDA)
- new net: C9.1, R14.2, U4.5 (VDD), U4.7 (SRN)
- new net BIN: U4.10 (BIN)
- new net GPOUT: U4.12 (GPOUT)
- new net VSYS: R14.1, U4.8 (SRP)
- no-connect marks 0 -> 3
