File: pg_hw/BMS.kicad_sch (KiCad schematic)
At the start: 14 parts, among them U4 BQ27441DRZR-G1A, U4 TP4056

Commit message: push
Parts:
- removed C6: 10uF, symbol Device:C
- removed C7: C, symbol Device:C
- removed D7, D8: LED, symbol Device:LED
- removed R10: 1K, Resistor_SMD:R_0402_1005Metric, symbol Device:R_US
- removed R11: RPROG, Resistor_SMD:R_0402_1005Metric, symbol Device:R_US
- removed R9: 1, Resistor_SMD:R_0402_1005Metric, symbol Device:R_US
- removed U4: TP4056, Package_SO:MSOP-8-1EP_3x3mm_P0.65mm_EP1.5x1.8mm, symbol ul_TP4056:TP4056
- added BT1: Battery, symbol Device:Battery
- R12, R13: value R_US -> 10K; footprint Resistor_SMD:R_0402_1005Metric -> (none)
Connections:
- net +5V is gone; now on net BIN: R13.1
- net VSYS is gone; now on net GND: R14.1, U4.8 (SRP)
- net GND: now also R13.2, BT1.1 (+), BT1.2 (-); no longer R12.2
- net GPOUT: now also R12.2
- net +3V3: now reaches R12.1
- net +3V3: no longer R13.2
- net VSYS_BMS: now reaches C9.1, R14.2, U4.5 (VDD), U4.7 (SRN)
Other:
- moved on the sheet: C10, C9, R14, U4

Commit message: adad
dada
Parts:
- C9: footprint Resistor_SMD:R_0603_1608Metric -> Capacitor_SMD:C_0603_1608Metric
- R12, R13: footprint (none) -> Resistor_SMD:R_0402_1005Metric
Changed lines of the file:
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@@
 			)
 		)
-		(property "Footprint" "Resistor_SMD:R_0603_1608Metric"
+		(property "Footprint" "Capacitor_SMD:C_0603_1608Metric"
 			(at 174.9552 95.25 0)
 			(effects
@@
 			)
 		)
-		(property "Footprint" ""
+		(property "Footprint" "Resistor_SMD:R_0402_1005Metric"
 			(at 110.236 57.404 90)
 			(effects
@@
 			)
 		)
-		(property "Footprint" ""
+		(property "Footprint" "Resistor_SMD:R_0402_1005Metric"
 			(at 106.426 91.694 90)
 			(effects

Commit message: Update BMS.kicad_sch
Connections:
- net GND: no longer BT1.1 (+), C10.1, R14.1, U4.6 (BAT), U4.8 (SRP)
- new net BAT+: BT1.1 (+), C10.1, R14.1, U4.6 (BAT), U4.8 (SRP)
Changed lines of the file:
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@@
-	)
-	(junction
-		(at 83.82 88.9)
-		(diameter 0)
-		(color 0 0 0 0)
 	)
 	(junction
@@
 	(wire
 		(pts
-			(xy 83.82 88.9) (xy 83.82 90.17)
+			(xy 83.82 82.55) (xy 83.82 90.17)
 		)
 		(stroke
@@
 	(wire
 		(pts
-			(xy 83.82 82.55) (xy 83.82 88.9)
-		)
-		(stroke
-			(width 0)
-			(type default)
-		)
-	)
-	(wire
-		(pts
 			(xy 128.27 76.2) (xy 111.76 76.2)
 		)
@@
 		(pts
 			(xy 166.37 96.52) (xy 166.37 99.06)
-		)
-		(stroke
-			(width 0)
-			(type default)
-		)
-	)
-	(wire
-		(pts
-			(xy 83.82 88.9) (xy 86.36 88.9)
 		)
 		(stroke
@@
 		(fields_autoplaced yes)
 		(effects
-			(font
-				(size 1.27 1.27)
-			)
-			(justify left bottom)
-		)
-	)
-	(label "PACKP"
-		(at 86.36 88.9 0)
-		(fields_autoplaced yes)
-		(effects
