File: pg_hw/pg_hw.kicad_pcb (KiCad board)
At the start: 2 copper layers, 114 x 84 mm, 0 parts

Commit message: adad
dada
Parts:
- added BZ1: Buzzer, Buzzer_Beeper:Buzzer_15x7.5RM7.6, F.Cu at (91.8, 105.6)
- added C1: 0.1uF, Capacitor_SMD:C_0603_1608Metric, B.Cu at (102.8, 58.1)
- added C10: 1uF, Capacitor_SMD:C_0603_1608Metric, B.Cu at (93.0, 63.9)
- added C11: 10uC, Capacitor_SMD:C_0603_1608Metric, B.Cu at (89.6, 86.7)
- added C12: C, Capacitor_SMD:C_0603_1608Metric, B.Cu at (134.0, 63.9)
- added C13: C, Capacitor_SMD:C_0603_1608Metric, B.Cu at (134.0, 66.4)
- added C14: C, Capacitor_SMD:C_0603_1608Metric, B.Cu at (134.0, 68.9)
- added C15: C, Capacitor_SMD:C_0603_1608Metric, B.Cu at (134.0, 71.4)
- added C16: C, Capacitor_SMD:C_0603_1608Metric, B.Cu at (134.0, 73.9)
- added C17: C, Capacitor_SMD:C_0603_1608Metric, B.Cu at (134.0, 76.4)
- added C18: C, Capacitor_SMD:C_0603_1608Metric, B.Cu at (134.0, 79.0)
- added C2: 10uF, Capacitor_SMD:C_0603_1608Metric, B.Cu at (102.8, 60.6)
- added C3: 10uF, Capacitor_SMD:C_0603_1608Metric, B.Cu at (102.8, 63.1)
- added C4: 0.1uF, Capacitor_SMD:C_0603_1608Metric, B.Cu at (102.8, 65.6)
- added C5: 1uF, Capacitor_SMD:C_0603_1608Metric, B.Cu at (102.8, 68.1)
- added C6: 10uF, Capacitor_SMD:C_0603_1608Metric, B.Cu at (95.8, 80.9)
- added C7: C, Capacitor_SMD:C_0603_1608Metric, B.Cu at (134.0, 61.4)
- added C8: 100nF, Capacitor_SMD:C_0603_1608Metric, B.Cu at (86.8, 81.8)
- added C9: 0.47uF, Capacitor_SMD:C_0603_1608Metric, B.Cu at (93.0, 61.4)
- added D1: SS14, Diode_SMD:D_SMA, B.Cu at (143.9, 62.4)
- added D2: ESD9B5.0ST5G, Diode_SMD:D_SOD-923, B.Cu at (114.4, 67.6)
- added D4: SS14, Diode_SMD:D_SMA, B.Cu at (143.9, 67.0)
- added D5: SS14, Diode_SMD:D_SMA, B.Cu at (143.9, 71.5)
- added D6: SS14, Diode_SMD:D_SMA, B.Cu at (155.3, 99.9)
- added D7: SS14, Diode_SMD:D_SMA, B.Cu at (165.9, 100.2)
- added D8: SS14, Diode_SMD:D_SMA, B.Cu at (152.0, 85.6)
- added D9: SS14, Diode_SMD:D_SMA, B.Cu at (115.6, 106.4)
- added J1: USB_B_Micro, Connector_USB:USB_Micro-B_Molex-105017-0001, F.Cu at (91.8, 132.2)
- added Q1: SS8050, Package_TO_SOT_SMD:SOT-23, B.Cu at (118.2, 61.0)
- added Q2: SS8050, Package_TO_SOT_SMD:SOT-23, B.Cu at (132.3, 82.7)
- added Q3: FS8205A, footprints:SOT-23-6L_TCP, B.Cu at (175.7, 78.3)
- added R10: 1K, Resistor_SMD:R_0402_1005Metric, B.Cu at (105.7, 82.4)
- added R11: 1.5K, Resistor_SMD:R_0402_1005Metric, B.Cu at (105.7, 84.4)
- added R12: 10K, Resistor_SMD:R_0402_1005Metric, B.Cu at (96.5, 61.1)
- added R13: 10K, Resistor_SMD:R_0402_1005Metric, B.Cu at (96.5, 63.1)
- added R14: 0.01, Resistor_SMD:R_0402_1005Metric, B.Cu at (96.5, 65.1)
- added R15: 1K, Resistor_SMD:R_0402_1005Metric, B.Cu at (105.7, 86.4)
- added R16: 100, Resistor_SMD:R_0402_1005Metric, B.Cu at (105.7, 88.4)
- added R17: R, Resistor_SMD:R_0402_1005Metric, B.Cu at (130.6, 61.1)
- added R18: R, Resistor_SMD:R_0402_1005Metric, B.Cu at (130.6, 63.1)
- added R19: R, Resistor_SMD:R_0402_1005Metric, B.Cu at (130.6, 65.1)
- added R20: R, Resistor_SMD:R_0402_1005Metric, B.Cu at (130.6, 67.1)
- added R21: R, Resistor_SMD:R_0402_1005Metric, B.Cu at (130.6, 69.1)
- added R22: R, Resistor_SMD:R_0402_1005Metric, B.Cu at (127.7, 61.1)
- added R23: R, Resistor_SMD:R_0402_1005Metric, B.Cu at (127.7, 63.1)
- added R24: R, Resistor_SMD:R_0402_1005Metric, B.Cu at (127.7, 65.1)
- added R27: 1K, Resistor_SMD:R_0402_1005Metric, B.Cu at (102.4, 82.9)
- added R28: 1K, Resistor_SMD:R_0402_1005Metric, B.Cu at (99.4, 85.1)
- added R29: 1K, Resistor_SMD:R_0402_1005Metric, B.Cu at (99.4, 87.1)
- added R3: 12K, Resistor_SMD:R_0402_1005Metric, B.Cu at (114.3, 59.6)
- added R30: 0, Resistor_SMD:R_0402_1005Metric, B.Cu at (111.4, 63.6)
- added R31: 0, Resistor_SMD:R_0402_1005Metric, B.Cu at (111.4, 65.6)
- added R32: 0, Resistor_SMD:R_0402_1005Metric, B.Cu at (108.5, 59.6)
- added R33: 0, Resistor_SMD:R_0402_1005Metric, B.Cu at (108.5, 61.6)
- added R34: 0, Resistor_SMD:R_0402_1005Metric, B.Cu at (108.5, 63.6)
- added R35: 10K, Resistor_SMD:R_0402_1005Metric, B.Cu at (108.5, 65.6)
- added R36: 1k, Resistor_SMD:R_0402_1005Metric, B.Cu at (127.7, 67.1)
- added R37: 0, Resistor_SMD:R_0402_1005Metric, B.Cu at (127.7, 69.1)
- added R4: 10K, Resistor_SMD:R_0402_1005Metric, B.Cu at (114.3, 61.6)
- added R5: 12K, Resistor_SMD:R_0402_1005Metric, B.Cu at (114.3, 63.6)
- added R6: 10K, Resistor_SMD:R_0402_1005Metric, B.Cu at (114.3, 65.6)
- added R7: 10K, Resistor_SMD:R_0402_1005Metric, B.Cu at (111.4, 59.6)
- added R8: 10K, Resistor_SMD:R_0402_1005Metric, B.Cu at (111.4, 61.6)
- added R9: 1, Resistor_SMD:R_0402_1005Metric, B.Cu at (99.9, 74.4)
- added U1: BW16, footprints:MODULE_BW16, B.Cu at (138.9, 120.7)
- added U2: AMS1117-3.3, Package_TO_SOT_SMD:SOT-223-3_TabPin2, B.Cu at (135.3, 94.4)
- added U3: CH340C, Package_SO:SOP-16_3.9x9.9mm_P1.27mm, B.Cu at (115.0, 124.3)
- added U5: TP4056, Package_SO:MSOP-8-1EP_3x3mm_P0.65mm_EP1.5x1.8mm, B.Cu at (168.4, 88.5)
- added U6: DW01A, Package_TO_SOT_SMD:SOT-23-6, B.Cu at (175.2, 84.2)
Other:
- board text added: "Celtiko"

Commit message: Update pg_hw.kicad_pcb
Parts:
- moved R14 22.2 mm to (113.2, 79.8)
- moved U3 22.1 mm to (92.9, 124.3), turned to 90 degrees
- moved U2 15.9 mm to (120.0, 90.0)
- moved R16 14.6 mm to (117.5, 79.8)
- moved U1 11.4 mm to (128.0, 123.7)
- moved J1 0.71 mm to (91.1, 132.3)
Changed lines of the file:
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@@
 	(footprint "Connector_USB:USB_Micro-B_Molex-105017-0001"
 		(layer "F.Cu")
-		(at 91.8 132.2)
+		(at 91.1 132.3)
 		(descr "http://www.molex.com/pdm_docs/sd/1050170001_sd.pdf")
 		(tags "Micro-USB SMD Typ-B")
@@
 	(footprint "Resistor_SMD:R_0402_1005Metric"
 		(layer "B.Cu")
-		(at 96.485 65.12 180)
+		(at 113.2 79.8 180)
 		(descr "Resistor SMD 0402 (1005 Metric), square (rectangular) end terminal, IPC_7351 nominal, (Body size source: IPC-SM-782 page 72, https://www.pcb-3d.com/wordpress/wp-content/uploads/ipc-sm-782a_amendment_1_and_2.pdf), generated with kicad-footprint-generator")
 		(tags "resistor")
@@
 	(footprint "Package_TO_SOT_SMD:SOT-223-3_TabPin2"
 		(layer "B.Cu")
-		(at 135.3 94.4 180)
+		(at 120 90 180)
 		(descr "module CMS SOT223 4 pins")
 		(tags "CMS SOT")
@@
 	(footprint "footprints:MODULE_BW16"
 		(layer "B.Cu")
-		(at 138.95 120.65 90)
+		(at 128 123.73175 90)
 		(property "Reference" "U1"
 			(at -6.175 -13.365 90)
@@
 	(footprint "Package_SO:SOP-16_3.9x9.9mm_P1.27mm"
 		(layer "B.Cu")
-		(at 115 124.3)
+		(at 92.9 124.3 90)
 		(descr "SOP, 16 Pin (https://www.diodes.com/assets/Datasheets/PAM8403.pdf), generated with kicad-footprint-generator ipc_gullwing_generator.py")
 		(tags "SOP SO")
 		(property "Reference" "U3"
-			(at 0 5.9 360)
+			(at 0 5.9 90)
 			(layer "B.SilkS")
 			(effects
@@
 		)
 		(property "Value" "CH340C"
-			(at 0 -5.9 360)
+			(at 0 -5.9 90)
 			(layer "B.Fab")
 			(effects
@@
 		)
 		(property "Footprint" "Package_SO:SOP-16_3.9x9.9mm_P1.27mm"
-			(at 0 0 360)
+			(at 0 0 90)
 			(layer "B.Fab")
 			(hide yes)
@@
 		)
 		(property "Datasheet" "https://datasheet.lcsc.com/szlcsc/Jiangsu-Qin-Heng-CH340C_C84681.pdf"
-			(at 0 0 360)
+			(at 0 0 90)
 			(layer "B.Fab")
 			(hide yes)
@@
 		)
 		(property "Description" "USB serial converter, crystal-less, UART, SOIC-16"
-			(at 0 0 360)
+			(at 0 0 90)
 			(layer "B.Fab")
 			(hide yes)
@@
 		(attr smd)
 		(fp_line
-			(start -1.95 -5.06)
+			(start 1.95 -5.06)
 			(end 0 -5.06)
 			(stroke
@@
 		)
 		(fp_line
-			(start -1.95 5.06)
-			(end 0 5.06)
+			(start -1.95 -5.06)
+			(end 0 -5.06)
 			(stroke
 				(width 0.12)
@@
 		)
 		(fp_line
-			(start 1.95 -5.06)
-			(end 0 -5.06)
+			(start 1.95 5.06)
+			(end 0 5.06)
 			(stroke
 				(width 0.12)
@@
 		)
 		(fp_line
-			(start 1.95 5.06)
+			(start -1.95 5.06)
 			(end 0 5.06)
 			(stroke
@@
 		)
 		(fp_line
-			(start -3.75 -5.2)
-			(end -3.75 5.2)
+			(start 3.75 -5.2)
+			(end -3.75 -5.2)
 			(stroke
 				(width 0.05)
@@
 		)
 		(fp_line
-			(start -3.75 5.2)
-			(end 3.75 5.2)
+			(start -3.75 -5.2)
+			(end -3.75 5.2)
 			(stroke
 				(width 0.05)
@@
 		)
 		(fp_line
-			(start 3.75 -5.2)
-			(end -3.75 -5.2)
+			(start 3.75 5.2)
+			(end 3.75 -5.2)
 			(stroke
 				(width 0.05)
@@
 		)
 		(fp_line
-			(start 3.75 5.2)
-			(end 3.75 -5.2)
+			(start -3.75 5.2)
+			(end 3.75 5.2)
 			(stroke
 				(width 0.05)
@@
 		)
 		(fp_line
-			(start -1.95 -4.95)
-			(end 1.95 -4.95)
+			(start 1.95 -4.95)
+			(end 1.95 4.95)
 			(stroke
 				(width 0.1)
@@
 		)
 		(fp_line
-			(start -1.95 3.975)
-			(end -1.95 -4.95)
+			(start -1.95 -4.95)
+			(end 1.95 -4.95)
 			(stroke
 				(width 0.1)
@@
 		)
 		(fp_line
-			(start -0.975 4.95)
-			(end -1.95 3.975)
+			(start -1.95 3.975)
+			(end -1.95 -4.95)
 			(stroke
 				(width 0.1)
@@
 		)
 		(fp_line
-			(start 1.95 -4.95)
-			(end 1.95 4.95)
+			(start 1.95 4.95)
+			(end -0.975 4.95)
 			(stroke
 				(width 0.1)
@@
 		)
 		(fp_line
-			(start 1.95 4.95)
-			(end -0.975 4.95)
+			(start -0.975 4.95)
+			(end -1.95 3.975)
 			(stroke
 				(width 0.1)
@@
 		)
 		(fp_text user "${REFERENCE}"
-			(at 0 0 360)
+			(at 0 0 90)
 			(layer "B.Fab")
 			(effects
@@
 		)
 		(pad "1" smd roundrect
-			(at -2.5 4.445)
+			(at -2.5 4.445 90)
 			(size 2 0.6)
 			(layers "B.Cu" "B.Paste" "B.Mask")
@@
 		)
 		(pad "2" smd roundrect
-			(at -2.5 3.175)
+			(at -2.5 3.175 90)
 			(size 2 0.6)
 			(layers "B.Cu" "B.Paste" "B.Mask")
@@
 		)
 		(pad "3" smd roundrect
-			(at -2.5 1.905)
+			(at -2.5 1.905 90)
 			(size 2 0.6)
 			(layers "B.Cu" "B.Paste" "B.Mask")
@@
 		)
 		(pad "4" smd roundrect
-			(at -2.5 0.635)
+			(at -2.5 0.635 90)
 			(size 2 0.6)
 			(layers "B.Cu" "B.Paste" "B.Mask")
@@
 		)
 		(pad "5" smd roundrect
-			(at -2.5 -0.635)
+			(at -2.5 -0.635 90)
 			(size 2 0.6)
 			(layers "B.Cu" "B.Paste" "B.Mask")
@@
 		)
 		(pad "6" smd roundrect
-			(at -2.5 -1.905)
+			(at -2.5 -1.905 90)
 			(size 2 0.6)
 			(layers "B.Cu" "B.Paste" "B.Mask")
@@
 		)
 		(pad "7" smd roundrect
-			(at -2.5 -3.175)
+			(at -2.5 -3.175 90)
 			(size 2 0.6)
 			(layers "B.Cu" "B.Paste" "B.Mask")
@@
 		)
 		(pad "8" smd roundrect
-			(at -2.5 -4.445)
+			(at -2.5 -4.445 90)
 			(size 2 0.6)
 			(layers "B.Cu" "B.Paste" "B.Mask")
@@
 		)
 		(pad "9" smd roundrect
-			(at 2.5 -4.445)
+			(at 2.5 -4.445 90)
 			(size 2 0.6)
 			(layers "B.Cu" "B.Paste" "B.Mask")
@@
 		)
 		(pad "10" smd roundrect
-			(at 2.5 -3.175)
+			(at 2.5 -3.175 90)
 			(size 2 0.6)
 			(layers "B.Cu" "B.Paste" "B.Mask")
@@
 		)
 		(pad "11" smd roundrect
-			(at 2.5 -1.905)
+			(at 2.5 -1.905 90)
 			(size 2 0.6)
 			(layers "B.Cu" "B.Paste" "B.Mask")
@@
 		)
 		(pad "12" smd roundrect
-			(at 2.5 -0.635)
+			(at 2.5 -0.635 90)
 			(size 2 0.6)
 			(layers "B.Cu" "B.Paste" "B.Mask")
@@
 		)
 		(pad "13" smd roundrect
-			(at 2.5 0.635)
+			(at 2.5 0.635 90)
 			(size 2 0.6)
 			(layers "B.Cu" "B.Paste" "B.Mask")
@@
 		)
 		(pad "14" smd roundrect
-			(at 2.5 1.905)
+			(at 2.5 1.905 90)
 			(size 2 0.6)
 			(layers "B.Cu" "B.Paste" "B.Mask")
@@
 		)
 		(pad "15" smd roundrect
-			(at 2.5 3.175)
+			(at 2.5 3.175 90)
 			(size 2 0.6)
 			(layers "B.Cu" "B.Paste" "B.Mask")
@@
 		)
 		(pad "16" smd roundrect
-			(at 2.5 4.445)
+			(at 2.5 4.445 90)
 			(size 2 0.6)
 			(layers "B.Cu" "B.Paste" "B.Mask")
@@
 	(footprint "Resistor_SMD:R_0402_1005Metric"
 		(layer "B.Cu")
-		(at 105.695476 88.4 180)
+		(at 117.5 79.8 180)
 		(descr "Resistor SMD 0402 (1005 Metric), square (rectangular) end terminal, IPC_7351 nominal, (Body size source: IPC-SM-782 page 72, https://www.pcb-3d.com/wordpress/wp-content/uploads/ipc-sm-782a_amendment_1_and_2.pdf), generated with kicad-footprint-generator")
 		(tags "resistor")
